Commit message: Initial Files

File: urdf/mech/base.urdf.xacro (robot description, xacro)
@@ -13,5 +13,8 @@
   <xacro:property name="torso_mass" value="10" />
   <!-- Elevator properties -->
-  <xacro:property name="elevator_length" value="0.02" />
+  <xacro:property name="elevator_length" value="0.03" />
+  <xacro:property name="elevator_width" value="0.12" />
+  <xacro:property name="elevator_height" value="0.62" />
+  <xacro:property name="elevator_distance" value="0.04" />
   <xacro:macro name="base">
     <link name="base_footprint"/>
@@ -92,5 +95,5 @@
         <origin xyz="0 0 0" rpy="0 0 0"/>
         <geometry>
-          <box size="${elevator_length} ${0.13} ${torso_height}"/>
+          <box size="${elevator_length} ${elevator_width} ${elevator_height}"/>
         </geometry>
         <material name="yellow">
@@ -115,5 +118,5 @@
       <parent link="torso_link"/>
       <child link="elevator_base_link"/>
-      <origin xyz="${torso_length/2 + elevator_length/2 - 0.01} 0 0" rpy="0 0 0"/>
+      <origin xyz="${torso_length/2 + elevator_length/2 - 0.01} 0 ${-elevator_distance}" rpy="0 0 0"/>
     </joint>
     <link name="elevator_part_link">
@@ -121,5 +124,5 @@
         <origin xyz="0 0 0" rpy="0 0 0"/>
         <geometry>
-          <box size="${0.01} ${0.13} ${0.13}"/>
+          <box size="${0.003} ${0.13} ${0.088}"/>
         </geometry>
         <material name="yellow">
@@ -130,5 +133,5 @@
         <origin xyz="0 0 0" rpy="0 0 0"/>
         <geometry>
-          <box size="${0.01} ${0.13} ${0.13}"/>
+          <box size="${0.003} ${0.13} ${0.088}"/>
         </geometry>
       </collision>
@@ -144,7 +147,7 @@
       <parent link="elevator_base_link"/>
       <child link="elevator_part_link"/>
-      <origin xyz="${elevator_length/2 + 0.005} 0 0" rpy="0 0 0"/>
+      <origin xyz="${elevator_length/2 + 0.00015} 0 0" rpy="0 0 0"/>
       <axis xyz="0 0 1"/>
-      <limit lower="${-torso_height/2 + 0.13/2}" upper="${torso_height/2 - 0.13/2}" effort="0.5" velocity="0.1"/>
+      <limit lower="${-elevator_height/2 + 0.088/2 + 0.012}" upper="${elevator_height/2 - 0.088/2 - 0.012}" effort="0.5" velocity="0.1"/>
     </joint>
   </xacro:macro>

File: urdf/robots/vera.urdf.xacro (robot description, xacro)
@@ -9,4 +9,6 @@
   <xacro:include filename="$(find vera_description)/urdf/controllers/omni_drive.urdf.xacro" />
   <xacro:include filename="$(find vera_description)/urdf/mech/manipulator.xml" />
+  <xacro:include filename="$(find vera_description)/urdf/utils/base.ros2_control.xacro" />
+  <xacro:include filename="$(find vera_description)/urdf/utils/manipulator.ros2_control.xacro" />
   <xacro:base/>
   <xacro:mecanum_wheel
@@ -49,4 +51,11 @@
   <xacro:elevator/>
   <xacro:manipulator/>
+  <xacro:manipulator_ros2_control
+    name="ManipulatorControl"
+    initial_positions_file="$(find vera_moveit_config)/config/initial_positions.yaml"
+  />
+  <!-- <xacro:base_ros2_control
+    name="BaseControl"
+  /> -->
   <!-- <xacro:imu/>
   <xacro:generic_laser>
